File: Metronome/Metronome.kicad_pcb (KiCad board)
At the start: 2 copper layers, 90.5 x 85 mm, 13 parts, among them J1 Conn_01x02_Pin, J2 Conn_01x02_Pin, J3 Conn_01x02_Pin, J4 Conn_01x04_Pin, J5 Conn_01x03_Pin, J6 Conn_01x05_Pin, U2 5V Buck_Conv, U4 TPA3110_AudioAmp

Commit message: Enclosure + Footprint Edits
Parts:
- R1, R2, R3: footprint Resistor_THT:R_Axial_DIN0204_L3.6mm_D1.6mm_P5.08mm_Horizontal -> Resistor_THT:R_Axial_DIN0204_L3.6mm_D1.6mm_P7.62mm_Horizontal
- moved J6 106.4 mm to (231.2, 147.6)
- moved U2 97.6 mm to (66.5, 69.8)
- moved R1 89.3 mm to (42.0, 91.8)
- moved R2 89.3 mm to (42.0, 97.3)
- moved R3 89.3 mm to (42.0, 102.8)
- moved J1 74.0 mm to (24.8, 135.8)
- moved J2 70.2 mm to (43.2, 170.2)
- moved U1 52.7 mm to (49.7, 134.8)
- moved J3 51.3 mm to (214.3, 133.2)
- moved J4 50.9 mm to (194.3, 150.2)
- moved J5 39.1 mm to (194.4, 135.4)
- moved A1 1.44 mm to (163.8, 118.8)
- moved U4 0.45 mm to (88.6, 122.4)
Connections:
- A1 pad 29: unconnected-(A1-GND-Pad29) -> GND
- A1 pad 4: unconnected-(A1-GND-Pad4) -> GND
Routing:
- net GND: track 164.8 -> 0.07 mm, vias 2 -> 0
- net +5V: track 139.4 -> 0.00 mm, vias 1 -> 0
- net Net-(A1-D9): track 95.6 -> 0.00 mm, vias 2 -> 0
- net /A0/BUSY: track 95.6 -> 0.00 mm
- net Net-(A1-D11): track 92.4 -> 0.00 mm, vias 3 -> 0
- net +9V: track 80.4 -> 0.00 mm
- net Net-(A1-D2): track 77.3 -> 0.00 mm, vias 3 -> 0
- net Net-(J3-SPK1): track 76.7 -> 0.00 mm
- net Net-(A1-A4): track 73.7 -> 0.00 mm
- net Net-(A1-D12): track 70.8 -> 0.00 mm, vias 2 -> 0
- net Net-(J3-SPK2): track 70.6 -> 0.00 mm
- net Net-(A1-A2): track 63.3 -> 0.00 mm, vias 1 -> 0
- net Net-(A1-D3): track 63.1 -> 0.00 mm, vias 2 -> 0
- net Net-(A1-A1): track 62.8 -> 0.00 mm, vias 2 -> 0
- net Net-(A1-A5): track 60.5 -> 0.00 mm, vias 1 -> 0
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- removed copper zone on B.Cu, net GND
- removed copper zone on F.Cu, net GND
Other:
- outline, holes or cut-outs redrawn
